Commit message: RViz controller is woring with twist keyboard

File: install/perceptron_robot_description/share/perceptron_robot_description/urdf/materials.xacro (robot description, xacro)
@@ -1 +1,6 @@
-/ros2_ws/perceptron/build/perceptron_robot_description/urdf/materials.xacro
+<?xml version="1.0" ?>
+<robot name="perceptron_robot" xmlns:xacro="http://www.ros.org/wiki/xacro" >
+<material name="silver">
+  <color rgba="0.700 0.700 0.700 1.000"/>
+</material>
+</robot>

File: install/perceptron_robot_description/share/perceptron_robot_description/urdf/perceptron_robot.xacro (robot description, xacro)
@@ -1 +1,266 @@
-/ros2_ws/perceptron/build/perceptron_robot_description/urdf/perceptron_robot.xacro
+<?xml version="1.0" ?>
+<robot name="perceptron_robot" xmlns:xacro="http://www.ros.org/wiki/xacro">
+<xacro:include filename="$(find perceptron_robot_description)/urdf/materials.xacro" />
+<xacro:include filename="$(find perceptron_robot_description)/urdf/perceptron_robot.trans" />
+<xacro:include filename="$(find perceptron_robot_description)/urdf/perceptron_robot.gazebo" />
+<link name="base_link">
+  <inertial>
+    <origin xyz="0.10235518948158412 0.15768644923066177 0.03531321960603257" rpy="0 0 0"/>
+    <mass value="5.28321629585233"/>
+    <inertia ixx="0.084731" iyy="0.132613" izz="0.201957" ixy="-0.000161" iyz="0.000101" ixz="-0.0"/>
+  </inertial>
+  <visual>
+    <origin xyz="0 0 0" rpy="0 0 0"/>
+    <geometry>
+      <mesh filename="package://perceptron_robot_description/meshes/base_link.stl" scale="0.001 0.001 0.001"/>
+    </geometry>
+    <material name="silver"/>
+  </visual>
+  <collision>
+    <origin xyz="0 0 0" rpy="0 0 0"/>
+    <geometry>
+      <mesh filename="package://perceptron_robot_description/meshes/base_link.stl" scale="0.001 0.001 0.001"/>
+    </geometry>
+  </collision>
+</link>
+<link name="rim_1_1">
+  <inertial>
+    <origin xyz="-1.4986378178705184e-07 0.0015115848240151789 -4.1318648651145207e-07" rpy="0 0 0"/>
+    <mass value="0.16214137289777292"/>
+    <inertia ixx="9e-05" iyy="0.000105" izz="9e-05" ixy="-0.0" iyz="0.0" ixz="-0.0"/>
+  </inertial>
+  <visual>
+    <origin xyz="-0.003148 0.040234 -0.032423" rpy="0 0 0"/>
+    <geometry>
+      <mesh filename="package://perceptron_robot_description/meshes/rim_1_1.stl" scale="0.001 0.001 0.001"/>
+    </geometry>
+    <material name="silver"/>
+  </visual>
+  <collision>
+    <origin xyz="-0.003148 0.040234 -0.032423" rpy="0 0 0"/>
+    <geometry>
+      <mesh filename="package://perceptron_robot_description/meshes/rim_1_1.stl" scale="0.001 0.001 0.001"/>
+    </geometry>
+  </collision>
+</link>
+<link name="rim_1_5">
+  <inertial>
+    <origin xyz="-2.269742116478568e-09 -0.008488317094600996 -2.73853864800333e-07" rpy="0 0 0"/>
+    <mass value="0.16214137289777292"/>
+    <inertia ixx="9e-05" iyy="0.000105" izz="9e-05" ixy="-0.0" iyz="0.0" ixz="-0.0"/>
+  </inertial>
+  <visual>
+    <origin xyz="-0.2191 0.035 -0.0314" rpy="0 0 0"/>
+    <geometry>
+      <mesh filename="package://perceptron_robot_description/meshes/rim_1_5.stl" scale="0.001 0.001 0.001"/>
+    </geometry>
+    <material name="silver"/>
+  </visual>
+  <collision>
+    <origin xyz="-0.2191 0.035 -0.0314" rpy="0 0 0"/>
+    <geometry>
+      <mesh filename="package://perceptron_robot_description/meshes/rim_1_5.stl" scale="0.001 0.001 0.001"/>
+    </geometry>
+  </collision>
+</link>
+<link name="rim_1_6">
+  <inertial>
+    <origin xyz="6.199178303502306e-09 0.008488317094601128 -2.73853864800333e-07" rpy="0 0 0"/>
+    <mass value="0.16214137289777292"/>
+    <inertia ixx="9e-05" iyy="0.000105" izz="9e-05" ixy="-0.0" iyz="-0.0" ixz="0.0"/>
+  </inertial>
+  <visual>
+    <origin xyz="-0.0051 -0.34 -0.0314" rpy="0 0 0"/>
+    <geometry>
+      <mesh filename="package://perceptron_robot_description/meshes/rim_1_6.stl" scale="0.001 0.001 0.001"/>
+    </geometry>
+    <material name="silver"/>
+  </visual>
+  <collision>
+    <origin xyz="-0.0051 -0.34 -0.0314" rpy="0 0 0"/>
+    <geometry>
+      <mesh filename="package://perceptron_robot_description/meshes/rim_1_6.stl" scale="0.001 0.001 0.001"/>
+    </geometry>
+  </collision>
+</link>
+<link name="rim_1_7">
+  <inertial>
+    <origin xyz="-2.2697420887229924e-09 0.008488317094601128 2.724501751774633e-07" rpy="0 0 0"/>
+    <mass value="0.16214137289777292"/>
+    <inertia ixx="9e-05" iyy="0.000105" izz="9e-05" ixy="0.0" iyz="0.0" ixz="0.0"/>
+  </inertial>
+  <visual>
+    <origin xyz="-0.2201 -0.34 -0.0314" rpy="0 0 0"/>
+    <geometry>
+      <mesh filename="package://perceptron_robot_description/meshes/rim_1_7.stl" scale="0.001 0.001 0.001"/>
+    </geometry>
+    <material name="silver"/>
+  </visual>
+  <collision>
+    <origin xyz="-0.2201 -0.34 -0.0314" rpy="0 0 0"/>
+    <geometry>
+      <mesh filename="package://perceptron_robot_description/meshes/rim_1_7.stl" scale="0.001 0.001 0.001"/>
+    </geometry>
+  </collision>
+</link>
+<link name="tyre_1">
+  <inertial>
+    <origin xyz="0.03140017357281477 -0.4827348354516158 -0.15699984818745197" rpy="0 0 0"/>
+    <mass value="0.5502920703903658"/>
+    <inertia ixx="0.00102" iyy="0.001663" izz="0.00102" ixy="0.0" iyz="0.0" ixz="-0.0"/>
+  </inertial>
+  <visual>
+    <origin xyz="-0.1877 -0.4406 -0.1884" rpy="0 0 0"/>
+    <geometry>
+      <mesh filename="package://perceptron_robot_description/meshes/tyre_1.stl" scale="0.001 0.001 0.001"/>
+    </geometry>
+    <material name="silver"/>
+  </visual>
+  <collision>
+    <origin xyz="-0.1877 -0.4406 -0.1884" rpy="0 0 0"/>
+    <geometry>
+      <mesh filename="package://perceptron_robot_description/meshes/tyre_1.stl" scale="0.001 0.001 0.001"/>
+    </geometry>
+  </collision>
+</link>
+<link name="tyre_5">
+  <inertial>
+    <origin xyz="0.032423025978775236 -0.6984812629814025 -0.12346598752007373" rpy="0 0 0"/>
+    <mass value="0.5502920703903658"/>
+    <inertia ixx="0.00102" iyy="0.001663" izz="0.00102" ixy="0.0" iyz="0.0" ixz="-0.0"/>
+  </inertial>
+  <visual>
+    <origin xyz="0.029275 -0.661318 -0.155889" rpy="0 0 0"/>
+    <geometry>
+      <mesh filename="package://perceptron_robot_description/meshes/tyre_5.stl" scale="0.001 0.001 0.001"/>
+    </geometry>
+    <material name="silver"/>
+  </visual>
+  <collision>
+    <origin xyz="0.029275 -0.661318 -0.155889" rpy="0 0 0"/>
+    <geometry>
+      <mesh filename="package://perceptron_robot_description/meshes/tyre_5.stl" scale="0.001 0.001 0.001"/>
+    </geometry>
+  </collision>
+</link>
+<link name="tyre_6">
+  <inertial>
+    <origin xyz="0.03140017357281516 0.4819006200792817 0.5043001518125478" rpy="0 0 0"/>
+    <mass value="0.5502920703903658"/>
+    <inertia ixx="0.00102" iyy="0.001663" izz="0.00102" ixy="0.0" iyz="0.0" ixz="-0.0"/>
+  </inertial>
+  <visual>
+    <origin xyz="-0.1887 0.1346 0.4729" rpy="0 0 0"/>
+    <geometry>
+      <mesh filename="package://perceptron_robot_description/meshes/tyre_6.stl" scale="0.001 0.001 0.001"/>
+    </geometry>
+    <material name="silver"/>
+  </visual>
+  <collision>
+    <origin xyz="-0.1887 0.1346 0.4729" rpy="0 0 0"/>
+    <geometry>
+      <mesh filename="package://perceptron_robot_description/meshes/tyre_6.stl" scale="0.001 0.001 0.001"/>
+    </geometry>
+  </collision>
+</link>
+<link name="tyre_7">
+  <inertial>
+    <origin xyz="-0.031399826427185265 0.6964006200792815 -0.504299848187452" rpy="0 0 0"/>
+    <mass value="0.5502920703903658"/>
+    <inertia ixx="0.00102" iyy="0.001663" izz="0.00102" ixy="0.0" iyz="0.0" ixz="-0.0"/>
+  </inertial>
+  <visual>
+    <origin xyz="-0.0365 0.3496 -0.5357" rpy="0 0 0"/>
+    <geometry>
+      <mesh filename="package://perceptron_robot_description/meshes/tyre_7.stl" scale="0.001 0.001 0.001"/>
+    </geometry>
+    <material name="silver"/>
+  </visual>
+  <collision>
+    <origin xyz="-0.0365 0.3496 -0.5357" rpy="0 0 0"/>
+    <geometry>
+      <mesh filename="package://perceptron_robot_description/meshes/tyre_7.stl" scale="0.001 0.001 0.001"/>
+    </geometry>
+  </collision>
+</link>
+<joint name="right_back" type="continuous">
+  <origin xyz="0.003148 -0.040234 0.032423" rpy="0 0 0"/>
+  <parent link="base_link"/>
+  <child link="rim_1_1"/>
+  <axis xyz="0.0 1.0 0.0"/>
+</joint>
+<joint name="right_front" type="continuous">
+  <origin xyz="0.2191 -0.035 0.0314" rpy="0 0 0"/>
+  <parent link="base_link"/>
+  <child link="rim_1_5"/>
+  <axis xyz="0.0 1.0 0.0"/>
+</joint>
+<joint name="left_back" type="continuous">
+  <origin xyz="0.0051 0.34 0.0314" rpy="0 0 0"/>
+  <parent link="base_link"/>
+  <child link="rim_1_6"/>
+  <axis xyz="0.0 1.0 0.0"/>
+</joint>
+<joint name="left_front" type="continuous">
+  <origin xyz="0.2201 0.34 0.0314" rpy="0 0 0"/>
+  <parent link="base_link"/>
+  <child link="rim_1_7"/>
+  <axis xyz="-0.0 1.0 0.0"/>
+</joint>
+<joint name="Rigid17" type="fixed">
+  <origin xyz="-0.0314 0.4756 0.157" rpy="0 0 0"/>
+  <parent link="rim_1_5"/>
+  <child link="tyre_1"/>
+</joint>
+<joint name="Rigid18" type="fixed">
+  <origin xyz="-0.032423 0.701552 0.123466" rpy="0 0 0"/>
+  <parent link="rim_1_1"/>
+  <child link="tyre_5"/>
+</joint>
+<joint name="Rigid19" type="fixed">
+  <origin xyz="-0.0314 -0.4746 -0.5043" rpy="0 0 0"/>
+  <parent link="rim_1_7"/>
+  <child link="tyre_6"/>
+</joint>
+<joint name="Rigid20" type="fixed">
+  <origin xyz="0.0314 -0.6896 0.5043" rpy="0 0 0"/>
+  <parent link="rim_1_6"/>
+  <child link="tyre_7"/>
+</joint>
+<!-- Add this block here for ros2_control with mock hardware -->
+<ros2_control name="GazeboSystem" type="system">
+  <hardware>
+    <plugin>mock_components/GenericSystem</plugin>
+    <!-- <plugin>gazebo_ros2_control/GazeboSystem</plugin> -->
+        <param name="calculate_dynamics">true</param>
+  </hardware>
+  <joint name="right_back">
+    <command_interface name="velocity"/>
+    <state_interface name="position">
+      <param name="initial_value">0.0</param>
+    </state_interface>
+    <state_interface name="velocity"/>
+  </joint>
+  <joint name="right_front">
+    <command_interface name="velocity"/>
+    <state_interface name="position">
+      <param name="initial_value">0.0</param>
+    </state_interface>
+    <state_interface name="velocity"/>
+  </joint>
+  <joint name="left_front">
+    <command_interface name="velocity"/>
+    <state_interface name="position">
+      <param name="initial_value">0.0</param>
+    </state_interface>
+    <state_interface name="velocity"/>
+  </joint>
+  <joint name="left_back">
+    <command_interface name="velocity"/>
+    <state_interface name="position">
+      <param name="initial_value">0.0</param>
+    </state_interface>
+    <state_interface name="velocity"/>
+  </joint>
+</ros2_control>
+</robot>
