Commit message: RViz controller is woring with twist keyboard

File: src/perceptron_robot_description/urdf/perceptron_robot.xacro (robot description, xacro)
@@ -2,11 +2,9 @@
 <robot name="perceptron_robot" xmlns:xacro="http://www.ros.org/wiki/xacro">
 <xacro:include filename="$(find perceptron_robot_description)/urdf/materials.xacro" />
-<xacro:include filename="$(find perceptron_robot_description)/urdf/perceptron_robot.trans" />
-<xacro:include filename="$(find perceptron_robot_description)/urdf/perceptron_robot.gazebo" />
 <link name="base_link">
   <inertial>
-    <origin xyz="0.15031355076933817 -0.20564481051841643 0.03531321960603249" rpy="0 0 0"/>
-    <mass value="5.283216295852332"/>
-    <inertia ixx="0.132613" iyy="0.084731" izz="0.201957" ixy="0.000161" iyz="-0.0" ixz="-0.000101"/>
+    <origin xyz="0.10235518948158412 0.15768644923066177 0.03531321960603257" rpy="0 0 0"/>
+    <mass value="5.28321629585233"/>
+    <inertia ixx="0.084731" iyy="0.132613" izz="0.201957" ixy="-0.000161" iyz="0.000101" ixz="-0.0"/>
   </inertial>
   <visual>
@@ -24,21 +22,81 @@
   </collision>
 </link>
-<link name="rim_1">
-  <inertial>
-    <origin xyz="0.007487843772255975 1.4220787850072192e-07 2.3373751312227853e-07" rpy="0 0 0"/>
-    <mass value="0.16214137289777972"/>
-    <inertia ixx="0.000105" iyy="9e-05" izz="9e-05" ixy="0.0" iyz="0.0" ixz="0.0"/>
-  </inertial>
-  <visual>
-    <origin xyz="-0.343 0.0889 -0.0314" rpy="0 0 0"/>
-    <geometry>
-      <mesh filename="package://perceptron_robot_description/meshes/rim_1.stl" scale="0.001 0.001 0.001"/>
-    </geometry>
-    <material name="silver"/>
-  </visual>
-  <collision>
-    <origin xyz="-0.343 0.0889 -0.0314" rpy="0 0 0"/>
-    <geometry>
-      <mesh filename="package://perceptron_robot_description/meshes/rim_1.stl" scale="0.001 0.001 0.001"/>
+<link name="rim_1_1">
+  <inertial>
+    <origin xyz="-1.4986378178705184e-07 0.0015115848240151789 -4.1318648651145207e-07" rpy="0 0 0"/>
+    <mass value="0.16214137289777292"/>
+    <inertia ixx="9e-05" iyy="0.000105" izz="9e-05" ixy="-0.0" iyz="0.0" ixz="-0.0"/>
+  </inertial>
+  <visual>
+    <origin xyz="-0.003148 0.040234 -0.032423" rpy="0 0 0"/>
+    <geometry>
+      <mesh filename="package://perceptron_robot_description/meshes/rim_1_1.stl" scale="0.001 0.001 0.001"/>
+    </geometry>
+    <material name="silver"/>
+  </visual>
+  <collision>
+    <origin xyz="-0.003148 0.040234 -0.032423" rpy="0 0 0"/>
+    <geometry>
+      <mesh filename="package://perceptron_robot_description/meshes/rim_1_1.stl" scale="0.001 0.001 0.001"/>
+    </geometry>
+  </collision>
+</link>
+<link name="rim_1_5">
+  <inertial>
+    <origin xyz="-2.269742116478568e-09 -0.008488317094600996 -2.73853864800333e-07" rpy="0 0 0"/>
+    <mass value="0.16214137289777292"/>
+    <inertia ixx="9e-05" iyy="0.000105" izz="9e-05" ixy="-0.0" iyz="0.0" ixz="-0.0"/>
+  </inertial>
+  <visual>
+    <origin xyz="-0.2191 0.035 -0.0314" rpy="0 0 0"/>
+    <geometry>
+      <mesh filename="package://perceptron_robot_description/meshes/rim_1_5.stl" scale="0.001 0.001 0.001"/>
+    </geometry>
+    <material name="silver"/>
+  </visual>
+  <collision>
+    <origin xyz="-0.2191 0.035 -0.0314" rpy="0 0 0"/>
+    <geometry>
+      <mesh filename="package://perceptron_robot_description/meshes/rim_1_5.stl" scale="0.001 0.001 0.001"/>
+    </geometry>
+  </collision>
+</link>
+<link name="rim_1_6">
+  <inertial>
+    <origin xyz="6.199178303502306e-09 0.008488317094601128 -2.73853864800333e-07" rpy="0 0 0"/>
+    <mass value="0.16214137289777292"/>
+    <inertia ixx="9e-05" iyy="0.000105" izz="9e-05" ixy="-0.0" iyz="-0.0" ixz="0.0"/>
+  </inertial>
+  <visual>
+    <origin xyz="-0.0051 -0.34 -0.0314" rpy="0 0 0"/>
+    <geometry>
+      <mesh filename="package://perceptron_robot_description/meshes/rim_1_6.stl" scale="0.001 0.001 0.001"/>
+    </geometry>
+    <material name="silver"/>
+  </visual>
+  <collision>
+    <origin xyz="-0.0051 -0.34 -0.0314" rpy="0 0 0"/>
+    <geometry>
+      <mesh filename="package://perceptron_robot_description/meshes/rim_1_6.stl" scale="0.001 0.001 0.001"/>
+    </geometry>
+  </collision>
+</link>
+<link name="rim_1_7">
+  <inertial>
+    <origin xyz="-2.2697420887229924e-09 0.008488317094601128 2.724501751774633e-07" rpy="0 0 0"/>
+    <mass value="0.16214137289777292"/>
+    <inertia ixx="9e-05" iyy="0.000105" izz="9e-05" ixy="0.0" iyz="0.0" ixz="0.0"/>
+  </inertial>
+  <visual>
+    <origin xyz="-0.2201 -0.34 -0.0314" rpy="0 0 0"/>
+    <geometry>
+      <mesh filename="package://perceptron_robot_description/meshes/rim_1_7.stl" scale="0.001 0.001 0.001"/>
+    </geometry>
+    <material name="silver"/>
+  </visual>
+  <collision>
+    <origin xyz="-0.2201 -0.34 -0.0314" rpy="0 0 0"/>
+    <geometry>
+      <mesh filename="package://perceptron_robot_description/meshes/rim_1_7.stl" scale="0.001 0.001 0.001"/>
     </geometry>
   </collision>
@@ -46,10 +104,10 @@
 <link name="tyre_1">
   <inertial>
-    <origin xyz="-0.022499378781032975 7.432448975719375e-08 -2.1858723067008645e-07" rpy="0 0 0"/>
-    <mass value="0.5502920703905811"/>
-    <inertia ixx="0.001663" iyy="0.00102" izz="0.00102" ixy="0.0" iyz="0.0" ixz="-0.0"/>
-  </inertial>
-  <visual>
-    <origin xyz="-0.373 0.0889 -0.0314" rpy="0 0 0"/>
+    <origin xyz="0.03140017357281477 -0.4827348354516158 -0.15699984818745197" rpy="0 0 0"/>
+    <mass value="0.5502920703903658"/>
+    <inertia ixx="0.00102" iyy="0.001663" izz="0.00102" ixy="0.0" iyz="0.0" ixz="-0.0"/>
+  </inertial>
+  <visual>
+    <origin xyz="-0.1877 -0.4406 -0.1884" rpy="0 0 0"/>
     <geometry>
       <mesh filename="package://perceptron_robot_description/meshes/tyre_1.stl" scale="0.001 0.001 0.001"/>
@@ -58,5 +116,5 @@
   </visual>
   <collision>
-    <origin xyz="-0.373 0.0889 -0.0314" rpy="0 0 0"/>
+    <origin xyz="-0.1877 -0.4406 -0.1884" rpy="0 0 0"/>
     <geometry>
       <mesh filename="package://perceptron_robot_description/meshes/tyre_1.stl" scale="0.001 0.001 0.001"/>
@@ -64,167 +122,143 @@
   </collision>
 </link>
-<link name="rim_2">
-  <inertial>
-    <origin xyz="0.008487941853639602 -1.413948607087434e-07 1.3311755303613282e-07" rpy="0 0 0"/>
-    <mass value="0.16214137289777972"/>
-    <inertia ixx="0.000105" iyy="9e-05" izz="9e-05" ixy="-0.0" iyz="-0.0" ixz="0.0"/>
-  </inertial>
-  <visual>
-    <origin xyz="-0.348234 0.304852 -0.032423" rpy="0 0 0"/>
-    <geometry>
-      <mesh filename="package://perceptron_robot_description/meshes/rim_2.stl" scale="0.001 0.001 0.001"/>
-    </geometry>
-    <material name="silver"/>
-  </visual>
-  <collision>
-    <origin xyz="-0.348234 0.304852 -0.032423" rpy="0 0 0"/>
-    <geometry>
-      <mesh filename="package://perceptron_robot_description/meshes/rim_2.stl" scale="0.001 0.001 0.001"/>
-    </geometry>
-  </collision>
-</link>
-<link name="tyre_2">
-  <inertial>
-    <origin xyz="-0.02249928069964946 2.5978772855150822e-08 -2.9254885998419855e-07" rpy="0 0 0"/>
-    <mass value="0.5502920703905811"/>
-    <inertia ixx="0.001663" iyy="0.00102" izz="0.00102" ixy="0.0" iyz="0.0" ixz="-0.0"/>
-  </inertial>
-  <visual>
-    <origin xyz="-0.379234 0.304852 -0.032423" rpy="0 0 0"/>
-    <geometry>
-      <mesh filename="package://perceptron_robot_description/meshes/tyre_2.stl" scale="0.001 0.001 0.001"/>
-    </geometry>
-    <material name="silver"/>
-  </visual>
-  <collision>
-    <origin xyz="-0.379234 0.304852 -0.032423" rpy="0 0 0"/>
-    <geometry>
-      <mesh filename="package://perceptron_robot_description/meshes/tyre_2.stl" scale="0.001 0.001 0.001"/>
-    </geometry>
-  </collision>
-</link>
-<link name="rim_3">
-  <inertial>
-    <origin xyz="-0.008487843772256011 6.199178836929775e-09 -2.7385386434236603e-07" rpy="0 0 0"/>
-    <mass value="0.16214137289777972"/>
-    <inertia ixx="0.000105" iyy="9e-05" izz="9e-05" ixy="0.0" iyz="0.0" ixz="0.0"/>
-  </inertial>
-  <visual>
-    <origin xyz="0.032 0.0879 -0.0314" rpy="0 0 0"/>
-    <geometry>
-      <mesh filename="package://perceptron_robot_description/meshes/rim_3.stl" scale="0.001 0.001 0.001"/>
-    </geometry>
-    <material name="silver"/>
-  </visual>
-  <collision>
-    <origin xyz="0.032 0.0879 -0.0314" rpy="0 0 0"/>
-    <geometry>
-      <mesh filename="package://perceptron_robot_description/meshes/rim_3.stl" scale="0.001 0.001 0.001"/>
-    </geometry>
-  </collision>
-</link>
-<link name="tyre_3">
-  <inertial>
-    <origin xyz="0.022500621218967072 1.7357281124896762e-07 -1.5321623789144034e-07" rpy="0 0 0"/>
-    <mass value="0.5502920703905811"/>
-    <inertia ixx="0.001663" iyy="0.00102" izz="0.00102" ixy="0.0" iyz="0.0" ixz="-0.0"/>
-  </inertial>
-  <visual>
-    <origin xyz="0.063 0.0879 -0.0314" rpy="0 0 0"/>
-    <geometry>
-      <mesh filename="package://perceptron_robot_description/meshes/tyre_3.stl" scale="0.001 0.001 0.001"/>
-    </geometry>
-    <material name="silver"/>
-  </visual>
-  <collision>
-    <origin xyz="0.063 0.0879 -0.0314" rpy="0 0 0"/>
-    <geometry>
-      <mesh filename="package://perceptron_robot_description/meshes/tyre_3.stl" scale="0.001 0.001 0.001"/>
-    </geometry>
-  </collision>
-</link>
-<link name="rim_4">
-  <inertial>
-    <origin xyz="-0.008487843772256087 6.199178725907473e-09 -2.738538642729771e-07" rpy="0 0 0"/>
-    <mass value="0.16214137289777972"/>
-    <inertia ixx="0.000105" iyy="9e-05" izz="9e-05" ixy="0.0" iyz="0.0" ixz="0.0"/>
-  </inertial>
-  <visual>
-    <origin xyz="0.032 0.3029 -0.0314" rpy="0 0 0"/>
-    <geometry>
-      <mesh filename="package://perceptron_robot_description/meshes/rim_4.stl" scale="0.001 0.001 0.001"/>
-    </geometry>
-    <material name="silver"/>
-  </visual>
-  <collision>
-    <origin xyz="0.032 0.3029 -0.0314" rpy="0 0 0"/>
-    <geometry>
-      <mesh filename="package://perceptron_robot_description/meshes/rim_4.stl" scale="0.001 0.001 0.001"/>
-    </geometry>
-  </collision>
-</link>
-<link name="tyre_4">
-  <inertial>
-    <origin xyz="-0.4661993787810331 -0.03139982642718875 0.1278998467837622" rpy="0 0 0"/>
-    <mass value="0.5502920703905811"/>
-    <inertia ixx="0.001663" iyy="0.00102" izz="0.00102" ixy="0.0" iyz="0.0" ixz="-0.0"/>
-  </inertial>
-  <visual>
-    <origin xyz="-0.42545 0.2715 0.0965" rpy="0 0 0"/>
-    <geometry>
-      <mesh filename="package://perceptron_robot_description/meshes/tyre_4.stl" scale="0.001 0.001 0.001"/>
-    </geometry>
-    <material name="silver"/>
-  </visual>
-  <collision>
-    <origin xyz="-0.42545 0.2715 0.0965" rpy="0 0 0"/>
-    <geometry>
-      <mesh filename="package://perceptron_robot_description/meshes/tyre_4.stl" scale="0.001 0.001 0.001"/>
-    </geometry>
-  </collision>
-</link>
-<joint name="Revolute_5" type="continuous">
-  <origin xyz="0.343 -0.0889 0.0314" rpy="0 0 0"/>
-  <parent link="base_link"/>
-  <child link="rim_1"/>
-  <axis xyz="1.0 0.0 0.0"/>
-</joint>
-<joint name="Rigid_6" type="fixed">
-  <origin xyz="0.03 0.0 0.0" rpy="0 0 0"/>
-  <parent link="rim_1"/>
+<link name="tyre_5">
+  <inertial>
+    <origin xyz="0.032423025978775236 -0.6984812629814025 -0.12346598752007373" rpy="0 0 0"/>
+    <mass value="0.5502920703903658"/>
+    <inertia ixx="0.00102" iyy="0.001663" izz="0.00102" ixy="0.0" iyz="0.0" ixz="-0.0"/>
+  </inertial>
+  <visual>
+    <origin xyz="0.029275 -0.661318 -0.155889" rpy="0 0 0"/>
+    <geometry>
+      <mesh filename="package://perceptron_robot_description/meshes/tyre_5.stl" scale="0.001 0.001 0.001"/>
+    </geometry>
+    <material name="silver"/>
+  </visual>
+  <collision>
+    <origin xyz="0.029275 -0.661318 -0.155889" rpy="0 0 0"/>
+    <geometry>
+      <mesh filename="package://perceptron_robot_description/meshes/tyre_5.stl" scale="0.001 0.001 0.001"/>
+    </geometry>
+  </collision>
+</link>
+<link name="tyre_6">
+  <inertial>
+    <origin xyz="0.03140017357281516 0.4819006200792817 0.5043001518125478" rpy="0 0 0"/>
+    <mass value="0.5502920703903658"/>
+    <inertia ixx="0.00102" iyy="0.001663" izz="0.00102" ixy="0.0" iyz="0.0" ixz="-0.0"/>
+  </inertial>
+  <visual>
+    <origin xyz="-0.1887 0.1346 0.4729" rpy="0 0 0"/>
+    <geometry>
+      <mesh filename="package://perceptron_robot_description/meshes/tyre_6.stl" scale="0.001 0.001 0.001"/>
+    </geometry>
+    <material name="silver"/>
+  </visual>
+  <collision>
+    <origin xyz="-0.1887 0.1346 0.4729" rpy="0 0 0"/>
+    <geometry>
+      <mesh filename="package://perceptron_robot_description/meshes/tyre_6.stl" scale="0.001 0.001 0.001"/>
+    </geometry>
+  </collision>
+</link>
+<link name="tyre_7">
+  <inertial>
+    <origin xyz="-0.031399826427185265 0.6964006200792815 -0.504299848187452" rpy="0 0 0"/>
+    <mass value="0.5502920703903658"/>
+    <inertia ixx="0.00102" iyy="0.001663" izz="0.00102" ixy="0.0" iyz="0.0" ixz="-0.0"/>
+  </inertial>
+  <visual>
+    <origin xyz="-0.0365 0.3496 -0.5357" rpy="0 0 0"/>
+    <geometry>
+      <mesh filename="package://perceptron_robot_description/meshes/tyre_7.stl" scale="0.001 0.001 0.001"/>
+    </geometry>
+    <material name="silver"/>
+  </visual>
+  <collision>
+    <origin xyz="-0.0365 0.3496 -0.5357" rpy="0 0 0"/>
+    <geometry>
+      <mesh filename="package://perceptron_robot_description/meshes/tyre_7.stl" scale="0.001 0.001 0.001"/>
+    </geometry>
+  </collision>
+</link>
+<joint name="right_back" type="continuous">
+  <origin xyz="0.003148 -0.040234 0.032423" rpy="0 0 0"/>
+  <parent link="base_link"/>
+  <child link="rim_1_1"/>
+  <axis xyz="0.0 1.0 0.0"/>
+</joint>
+<joint name="right_front" type="continuous">
+  <origin xyz="0.2191 -0.035 0.0314" rpy="0 0 0"/>
+  <parent link="base_link"/>
+  <child link="rim_1_5"/>
+  <axis xyz="0.0 1.0 0.0"/>
+</joint>
+<joint name="left_back" type="continuous">
+  <origin xyz="0.0051 0.34 0.0314" rpy="0 0 0"/>
+  <parent link="base_link"/>
+  <child link="rim_1_6"/>
+  <axis xyz="0.0 1.0 0.0"/>
+</joint>
+<joint name="left_front" type="continuous">
+  <origin xyz="0.2201 0.34 0.0314" rpy="0 0 0"/>
+  <parent link="base_link"/>
+  <child link="rim_1_7"/>
+  <axis xyz="-0.0 1.0 0.0"/>
+</joint>
+<joint name="Rigid17" type="fixed">
+  <origin xyz="-0.0314 0.4756 0.157" rpy="0 0 0"/>
+  <parent link="rim_1_5"/>
   <child link="tyre_1"/>
 </joint>
-<joint name="Revolute_7" type="continuous">
-  <origin xyz="0.348234 -0.304852 0.032423" rpy="0 0 0"/>
-  <parent link="base_link"/>
-  <child link="rim_2"/>
-  <axis xyz="1.0 0.0 0.0"/>
-</joint>
-<joint name="Rigid_8" type="fixed">
-  <origin xyz="0.031 0.0 0.0" rpy="0 0 0"/>
-  <parent link="rim_2"/>
-  <child link="tyre_2"/>
-</joint>
-<joint name="Revolute_9" type="continuous">
-  <origin xyz="-0.032 -0.0879 0.0314" rpy="0 0 0"/>
-  <parent link="base_link"/>
-  <child link="rim_3"/>
-  <axis xyz="-1.0 0.0 0.0"/>
-</joint>
-<joint name="Rigid_10" type="fixed">
-  <origin xyz="-0.031 0.0 0.0" rpy="0 0 0"/>
-  <parent link="rim_3"/>
-  <child link="tyre_3"/>
-</joint>
-<joint name="Revolute_11" type="continuous">
-  <origin xyz="-0.032 -0.3029 0.0314" rpy="0 0 0"/>
-  <parent link="base_link"/>
-  <child link="rim_4"/>
-  <axis xyz="-1.0 0.0 0.0"/>
-</joint>
-<joint name="Rigid_12" type="fixed">
-  <origin xyz="0.45745 0.0314 -0.1279" rpy="0 0 0"/>
-  <parent link="rim_4"/>
-  <child link="tyre_4"/>
-</joint>
+<joint name="Rigid18" type="fixed">
+  <origin xyz="-0.032423 0.701552 0.123466" rpy="0 0 0"/>
+  <parent link="rim_1_1"/>
+  <child link="tyre_5"/>
+</joint>
+<joint name="Rigid19" type="fixed">
+  <origin xyz="-0.0314 -0.4746 -0.5043" rpy="0 0 0"/>
+  <parent link="rim_1_7"/>
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