Commit message: everything upto controllers and gazebo and rivz is working.....

File: install/perceptron_robot_description/share/perceptron_robot_description/urdf/perceptron_robot.xacro (robot description, xacro)
@@ -5,4 +5,5 @@
 <xacro:arg name="is_sim" default="true"/>
 <xacro:arg name="gazebo_controllers" default="$(find perceptron_robot_control)/config/controllers.yaml"/>
+<xacro:property name="pkg_desc" value="$(find-pkg-share perceptron_robot_description)" />
 <link name="base_link">
   <inertial>
